Commit message: Add gr1t1 xml (attention urdf compile setting)

File: resources/robots/gr1t1/urdf/gr1t1_12dof.urdf (robot description, URDF)
Before this commit: robot gr1t2, 71 links, 70 joints
Links:
- added link world
- link L_hand_base_link: geometry collision mesh filename=../meshes/L_hand_base_link.STL; visual mesh filename=../meshes/L_hand_base_link.STL
- link L_index_intermediate_link: geometry collision mesh filename=../meshes/L_index_intermediate_link.STL; visual mesh filename=../meshes/L_index_intermediate_link.STL
- link L_index_proximal_link: geometry collision mesh filename=../meshes/L_index_proximal_link.STL; visual mesh filename=../meshes/L_index_proximal_link.STL
- link L_middle_intermediate_link: geometry collision mesh filename=../meshes/L_middle_intermediate_link.STL; visual mesh filename=../meshes/L_middle_intermediate_link.STL
- link L_middle_proximal_link: geometry collision mesh filename=../meshes/L_middle_proximal_link.STL; visual mesh filename=../meshes/L_middle_proximal_link.STL
- link L_pinky_intermediate_link: geometry collision mesh filename=../meshes/L_pinky_intermediate_link.STL; visual mesh filename=../meshes/L_pinky_intermediate_link.STL
- link L_pinky_proximal_link: geometry collision mesh filename=../meshes/L_pinky_proximal_link.STL; visual mesh filename=../meshes/L_pinky_proximal_link.STL
- link L_ring_intermediate_link: geometry collision mesh filename=../meshes/L_ring_intermediate_link.STL; visual mesh filename=../meshes/L_ring_intermediate_link.STL
- link L_ring_proximal_link: geometry collision mesh filename=../meshes/L_ring_proximal_link.STL; visual mesh filename=../meshes/L_ring_proximal_link.STL
- link L_thumb_distal_link: geometry collision mesh filename=../meshes/L_thumb_distal_link.STL; visual mesh filename=../meshes/L_thumb_distal_link.STL
- link L_thumb_proximal_pitch_link: geometry collision mesh filename=../meshes/L_thumb_proximal_pitch_link.STL; visual mesh filename=../meshes/L_thumb_proximal_pitch_link.STL
- link L_thumb_proximal_yaw_link: geometry collision mesh filename=../meshes/L_thumb_proximal_yaw_link.STL; visual mesh filename=../meshes/L_thumb_proximal_yaw_link.STL
- link R_hand_base_link: geometry collision mesh filename=../meshes/R_hand_base_link.STL; visual mesh filename=../meshes/R_hand_base_link.STL
- link R_index_intermediate_link: geometry collision mesh filename=../meshes/R_index_intermediate_link.STL; visual mesh filename=../meshes/R_index_intermediate_link.STL
- link R_index_proximal_link: geometry collision mesh filename=../meshes/R_index_proximal_link.STL; visual mesh filename=../meshes/R_index_proximal_link.STL
- link R_middle_intermediate_link: geometry collision mesh filename=../meshes/R_middle_intermediate_link.STL; visual mesh filename=../meshes/R_middle_intermediate_link.STL
- link R_middle_proximal_link: geometry collision mesh filename=../meshes/R_middle_proximal_link.STL; visual mesh filename=../meshes/R_middle_proximal_link.STL
- link R_pinky_intermediate_link: geometry collision mesh filename=../meshes/R_pinky_intermediate_link.STL; visual mesh filename=../meshes/R_pinky_intermediate_link.STL
- link R_pinky_proximal_link: geometry collision mesh filename=../meshes/R_pinky_proximal_link.STL; visual mesh filename=../meshes/R_pinky_proximal_link.STL
- link R_ring_intermediate_link: geometry collision mesh filename=../meshes/R_ring_intermediate_link.STL; visual mesh filename=../meshes/R_ring_intermediate_link.STL
- link R_ring_proximal_link: geometry collision mesh filename=../meshes/R_ring_proximal_link.STL; visual mesh filename=../meshes/R_ring_proximal_link.STL
- link R_thumb_distal_link: geometry collision mesh filename=../meshes/R_thumb_distal_link.STL; visual mesh filename=../meshes/R_thumb_distal_link.STL
- link R_thumb_proximal_pitch_link: geometry collision mesh filename=../meshes/R_thumb_proximal_pitch_link.STL; visual mesh filename=../meshes/R_thumb_proximal_pitch_link.STL
- link R_thumb_proximal_yaw_link: geometry collision mesh filename=../meshes/R_thumb_proximal_yaw_link.STL; visual mesh filename=../meshes/R_thumb_proximal_yaw_link.STL
Joints:
- added joint floating_base_joint: type floating, parent world, child base_link
